File: KiCad-Project/Joystick-Tester.kicad_pcb (KiCad board)
At the start: 2 copper layers, 35 x 44 mm, 9 parts, among them J1 DB9_Female

Commit message: Adding my company logo and silk screen info to PCB
Parts:
- added G***: LOGO, ShiroLogo:ShiroLogo, B.Cu at (155.0, 57.5)
Other:
- board text added: "Atari / Commodore / Amiga Joystick Tester V1.0"
- board text removed: "shiro.com.au Atari / Commodore / Amiga Joystick tester v 1.0"
